File: eagle/BootSel-Atmega.sch (EAGLE design)
At the start: 8 parts, among them Q1 20MHz

Commit message: smaller changes
Parts:
- added R1: 270R, resistor:R-EU_0204/5
Connections:
- net CIA34 renamed /CIA_RESET
- new net N$1: MEGA.PB7(XTAL2/TOSC2), R1.2
- net N$16: now also R1.1; no longer MEGA.PB7(XTAL2/TOSC2)
Other:
- note added: "/SEL0"
- note added: "/SEL1"
- note added: "/SEL2"
- note added: "/SEL3"
- moved on the sheet: C1, C2, MODE, Q1

Commit message: Fixed ISP connecotor.
Connections:
- removed net ISP_RST: BOARD.16, ISP.5, MEGA.PB2(SS/OC1B)
- new net /ISP_RST: ISP.5, MEGA.PC6(/RESET)
- new net /SEL3: BOARD.16, MEGA.PB2(SS/OC1B)
Changed lines of the file:
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@@
 </segment>
 </net>
-<net name="ISP_RST" class="0">
-<segment>
-<pinref part="ISP" gate="B" pin="5"/>
+<net name="/SEL3" class="0">
+<segment>
 <pinref part="MEGA" gate="G$1" pin="PB2(SS/OC1B)"/>
-<wire x1="53.34" y1="27.94" x2="53.34" y2="12.7" width="0.1524" layer="91"/>
-<wire x1="53.34" y1="12.7" x2="38.1" y2="12.7" width="0.1524" layer="91"/>
 <pinref part="BOARD" gate="G$1" pin="16"/>
 <wire x1="38.1" y1="12.7" x2="-25.4" y2="12.7" width="0.1524" layer="91"/>
 <wire x1="63.5" y1="-58.42" x2="38.1" y2="-58.42" width="0.1524" layer="91"/>
 <wire x1="38.1" y1="-58.42" x2="38.1" y2="12.7" width="0.1524" layer="91"/>
-<junction x="38.1" y="12.7"/>
 <label x="-5.08" y="12.7" size="1.778" layer="95"/>
 </segment>
@@
 </segment>
 </net>
+<net name="/ISP_RST" class="0">
+<segment>
+<pinref part="MEGA" gate="G$1" pin="PC6(/RESET)"/>
+<wire x1="-73.66" y1="63.5" x2="-73.66" y2="71.12" width="0.1524" layer="91"/>
+<wire x1="-73.66" y1="71.12" x2="22.86" y2="71.12" width="0.1524" layer="91"/>
+<wire x1="22.86" y1="71.12" x2="22.86" y2="25.4" width="0.1524" layer="91"/>
+<wire x1="22.86" y1="25.4" x2="53.34" y2="25.4" width="0.1524" layer="91"/>
+<pinref part="ISP" gate="B" pin="5"/>
+<wire x1="53.34" y1="25.4" x2="53.34" y2="27.94" width="0.1524" layer="91"/>
+<label x="25.4" y="25.4" size="1.778" layer="95"/>
+<label x="-33.02" y="68.58" size="1.778" layer="95"/>
+</segment>
+</net>
