File: eagle/JSchoenfeld-TTL-Version/Bootselector.sch (EAGLE design)
At the start: 10 parts, among them IC3 74HC00N, IC4 74HC157N

Commit message: 0.96
Parts:
- removed CFG: (no value), jumper:JP4Q
- added SJ1, SJ2, SJ3, SJ4: (no value), jumper:SJ
- TRIGGER: value 1-2=KS<2.0 -> (none); device jumper:JP2E -> jumper:SJ2W
- renumbered A500 to BRD
Connections:
- net N$7 renamed TRG
- net N$8 renamed SELENABLE
- net TRIGGER renamed /TRGSEL
- removed net /NEW_SELX: CFG.1, CFG.7, IC4A.2Y
- new net /NEWSELX: IC4A.2Y, SJ1.2, SJ4.2
- new net /SEL3: CIAG$1.PB6, TRIGGER.1
- net /NEWSEL1: now also SJ2.2; no longer CFG.5
- net /NEWSEL2: now also SJ3.2; no longer CFG.3
- net /SEL0: now also TRIGGER.3; no longer TRIGGER.1
- net /SEL1: now also SJ2.1; no longer CFG.6
- net /SEL2: now also SJ3.1; no longer CFG.4
- net /SELX: now also SJ1.1, SJ4.1; no longer CFG.2, CFG.8
- net PB6: no longer CIAG$1.PB6, TRIGGER.3
Other:
- moved on the sheet: C1, IC4P

Commit message: smaller changes
Connections:
- removed net PB6: BRDG$1.PB6
- net /SEL3: now also BRDG$1.PB6
Changed lines of the file:
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@@
-</segment>
-</net>
-<net name="PB6" class="0">
-<segment>
-<pinref part="BRD" gate="G$1" pin="PB6"/>
-<wire x1="58.42" y1="33.02" x2="68.58" y2="33.02" width="0.1524" layer="91"/>
-<wire x1="71.12" y1="35.56" x2="68.58" y2="33.02" width="0.1524" layer="91"/>
 </segment>
 </net>
@@
 <pinref part="TRIGGER" gate="G$1" pin="1"/>
 </segment>
-</net>
+<segment>
+<pinref part="BRD" gate="G$1" pin="PB6"/>
+<wire x1="58.42" y1="33.02" x2="68.58" y2="33.02" width="0.1524" layer="91"/>
+<wire x1="71.12" y1="35.56" x2="68.58" y2="33.02" width="0.1524" layer="91"/>
+</segment>
+</net>
