File: JSchoenfeld-TTL-Version/eagle/Boot_selector_SMD.sch (EAGLE design)
At the start: 12 parts, among them IC3 74HC00N, IC4 74HC157N

Commit message: Changes by 'e5frog' - SMT version, updated THT version.
Parts:
- removed CIA: CIA_DIP, Amiga:CIA_DIP
- removed DISABLE: (no value), jumper:JP1E
- removed SJX: (no value), jumper:SJ
- added ENABLE: on/off, jumper:JP1E
- added SJ3, SJ4: (no value), jumper:SJ
- added SOCKET: CIA_DIP, Amiga:CIA_DIP
- BRD: value CIA_DIP -> PINS
- C1: device rcl:C-EU050-025X075 -> rcl:C-EUC0805
- C2: device rcl:C-EU050-025X075 -> rcl:C-EUC0805K
- IC3: value 74HC00N -> 74HCT00D; device 74xx-eu:74HC00N -> 74xx-eu:74HCT00D
- IC4: value 74HC157N -> 74HCT157D; device 74xx-eu:74HC157N -> 74xx-eu:74HCT157D
- R1: device rcl:R-EU_0204/7 -> rcl:R-EU_R0805
Connections:
- net /NEWSEL0 renamed !NEWSEL0
- net SELENABLE renamed SEL_ENABLE
- removed net /NEWSEL1: BRDG$1.PB4, SJ1.2
- removed net /NEWSEL2: BRDG$1.PB5, SJ2.2
- removed net /NEWSELX: IC4A.2Y, SJX.2
- removed net /SEL0: CIAG$1.PB3, IC4A.1A, IC4A.2B, TRIGGER.3
- removed net /SEL1: CIAG$1.PB4, SJ1.1
- removed net /SEL2: CIAG$1.PB5, SJ2.1
- removed net /SEL3: BRDG$1.PB6, CIAG$1.PB6, TRIGGER.1
- removed net /SELX: IC4A.1B, IC4A.2A, SJX.1
- new net !NEWSEL1: BRDG$1.PB4, SJ2.2
- new net !NEWSEL2: BRDG$1.PB5, SJ3.2
- new net !NEWSELX: IC4A.2Y, SJ1.2, SJ4.2
- new net !SEL0: IC4A.1A, IC4A.2B, SOCKETG$1.PB3, TRIGGER.3
- new net !SEL1: SJ2.1, SOCKETG$1.PB4
- new net !SEL2: SJ3.1, SOCKETG$1.PB5
- new net !SEL3: BRDG$1.PB6, SOCKETG$1.PB6, TRIGGER.1
- new net !SELX: IC4A.1B, IC4A.2A, SJ1.1, SJ4.1
- net C: now also SOCKETG$1.C; no longer CIAG$1.C
- net CS: now also SOCKETG$1.!CS; no longer CIAG$1.!CS
- net D0: now also SOCKETG$1.D0; no longer CIAG$1.D0
- net D1: now also SOCKETG$1.D1; no longer CIAG$1.D1
- net D2: now also SOCKETG$1.D2; no longer CIAG$1.D2
- net D3: now also SOCKETG$1.D3; no longer CIAG$1.D3
- net D4: now also SOCKETG$1.D4; no longer CIAG$1.D4
- net D5: now also SOCKETG$1.D5; no longer CIAG$1.D5
- net D6: now also SOCKETG$1.D6; no longer CIAG$1.D6
- net D7: now also SOCKETG$1.D7; no longer CIAG$1.D7
- net E: now also SOCKETG$1.E; no longer CIAG$1.E
- net F: now also SOCKETG$1.!F; no longer CIAG$1.!F
- net GND: now also ENABLE.2, SOCKETPWR.GND1; no longer CIAPWR.GND1, DISABLE.2
- net INT: now also SOCKETG$1.!INT; no longer CIAG$1.!INT
- net N$2: now also ENABLE.1; no longer DISABLE.1
- net PA0: now also SOCKETG$1.PA0; no longer CIAG$1.PA0
- net PA1: now also SOCKETG$1.PA1; no longer CIAG$1.PA1
- net PA2: now also SOCKETG$1.PA2; no longer CIAG$1.PA2
- net PA3: now also SOCKETG$1.PA3; no longer CIAG$1.PA3
- net PA4: now also SOCKETG$1.PA4; no longer CIAG$1.PA4
- net PA5: now also SOCKETG$1.PA5; no longer CIAG$1.PA5
- net PA6: now also SOCKETG$1.PA6; no longer CIAG$1.PA6
- net PA7: now also SOCKETG$1.PA7; no longer CIAG$1.PA7
- net PB0: now also SOCKETG$1.PB0; no longer CIAG$1.PB0
- net PB1: now also SOCKETG$1.PB1; no longer CIAG$1.PB1
- net PB2: now also SOCKETG$1.PB2; no longer CIAG$1.PB2
- net PB7: now also SOCKETG$1.PB7; no longer CIAG$1.PB7
- net PC: now also SOCKETG$1.!PC; no longer CIAG$1.!PC
- net RESET: now also SOCKETG$1.!RESET; no longer CIAG$1.!RESET
- net RS0: now also SOCKETG$1.RS0; no longer CIAG$1.RS0
- net RS1: now also SOCKETG$1.RS1; no longer CIAG$1.RS1
- net RS2: now also SOCKETG$1.RS2; no longer CIAG$1.RS2
- net RS3: now also SOCKETG$1.RS3; no longer CIAG$1.RS3
- net S: now also SOCKETG$1.S; no longer CIAG$1.S
- net TICK: now also SOCKETG$1.TICK; no longer CIAG$1.TICK
- net VCC: now also SOCKETPWR.VCC1; no longer CIAPWR.VCC1
- net W: now also SOCKETG$1.!W; no longer CIAG$1.!W
Other:
- moved on the sheet: BRDPWR, C1, C2, IC3A, IC3B, IC3C, IC3D, IC3P, IC4, IC4P, R1, SJ1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
