File: JSchoenfeld-TTL-Version/eagle/Bootselector.brd (EAGLE design)
At the start: 22 x 55.2 mm, 13 parts, among them IC3 74HC00N, IC4 74HC157N

Commit message: Changes by 'e5frog' - SMT version, updated THT version.
Parts:
- removed SJ3, SJ4: (no value), jumper:SJ
- added SJX: (no value), jumper:SJ
- R1: value 10K -> 10k; device rcl:0207/10 -> rcl:0204/7
- moved SJ2 3.00 mm to (11.0, 16.0)
- moved IC4 1.04 mm to (11.2, 40.6)
- moved SJ1 1.00 mm to (11.0, 20.0)
- renumbered ENABLE to DISABLE
Connections:
- net /NEWSEL1: now also SJ1.2; no longer SJ2.2
- net /NEWSEL2: now also SJ2.2; no longer SJ3.2
- net /NEWSELX: now also SJX.2; no longer SJ1.2, SJ4.2
- net /SEL1: now also SJ1.1; no longer SJ2.1
- net /SEL2: now also SJ2.1; no longer SJ3.1
- net /SELX: now also SJX.1; no longer SJ1.1, SJ4.1
- net GND: now also IC4.10, IC4.11, IC4.13, IC4.14
Routing:
- net /SEL0: track 51.0 -> 61.1 mm
- net /NEWSEL0: track 20.3 -> 28.4 mm
- net VCC: track 70.9 -> 78.3 mm
- net SELENABLE: track 49.2 -> 56.0 mm
- net /NEWSELX: track 30.4 -> 23.8 mm, vias 0 -> 1
- net RESET: track 24.1 -> 30.8 mm
- net /SELX: track 39.4 -> 34.6 mm
- net N$2: track 28.1 -> 31.3 mm
- net TRG: track 8.67 -> 10.1 mm
- net /SEL3: track 12.3 -> 12.9 mm
Other:
- board text added: "(c) J. Schoenfeld - www.c64.de Artwork by o.eschi/moette/e5frog"
- board text removed: "(c) J. Schoenfeld - www.c64.de Artwork by o.eschi / moette"
